Commit message: Updating urdf and servos configuration

File: widowx_arm_description/urdf/widowx.urdf.xacro (robot description, xacro)
@@ -212,12 +212,12 @@
          <child link="${prefix}biceps_link" />
          <axis xyz="0 1 0" />
-         <limit lower="-1.575" upper="1.575" effort="0" velocity="1.571" />
+         <limit lower="-1.571" upper="1.571" effort="0" velocity="1.571" />
       </joint>
       <joint name="${prefix}joint_3" type="revolute">
-         <origin xyz="${M_SCALE*48.25} 0 ${M_SCALE*142.03}" rpy="0 0 0" />
+         <origin xyz="${M_SCALE*48.25} 0 ${M_SCALE*142.03}" rpy="0 ${M_PI/2.0} 0" />
          <parent link="${prefix}biceps_link" />
          <child link="${prefix}forearm_link" />
          <axis xyz="0 1 0" />
-         <limit lower="0" upper="2.617" effort="0" velocity="1.571" />
+         <limit lower="-1.571" upper="1.571" effort="0" velocity="1.571" />
       </joint>
       <joint name="${prefix}joint_4" type="revolute">

Commit message: Added python node and arm.yaml modified

File: widowx_arm_description/urdf/widowx.urdf.xacro (robot description, xacro)
@@ -246,5 +246,5 @@
          <parent link="${prefix}gripper_rail_link" />
          <child link="${prefix}gripper_1_link" />
-         <axis xyz="0 -1 0" />
+         <axis xyz="0 1 0" />
          <limit lower="0" upper="0.027" effort="0" velocity="0.5" />
       </joint>
@@ -254,5 +254,5 @@
          <child link="${prefix}gripper_2_link" />
          <mimic joint="${prefix}joint_7" />
-         <axis xyz="0 1 0" />
+         <axis xyz="0 -1 0" />
          <limit lower="0" upper="0.027" effort="0" velocity="0.5" />
       </joint>

Commit message: Added node to control the gripper

File: widowx_arm_description/urdf/widowx.urdf.xacro (robot description, xacro)
@@ -153,4 +153,6 @@
          </inertial>
       </link>
+      <link name="${prefix}gripper_aux_link">
+      </link>
       <link name="${prefix}gripper_1_link">
          <visual>
@@ -242,17 +244,24 @@
          <limit lower="-0.31" upper="0.1" effort="0" velocity="0.5" />
       </joint>
-      <joint name="${prefix}joint_7" type="prismatic">
+      <joint name="${prefix}gripper_revolute_joint" type="revolute">
+         <origin xyz = "0 0 0" rpy="0 0 0" />
+         <parent link="${prefix}gripper_rail_link" />
+         <child link="${prefix}gripper_aux_link" />
+         <axis xyz="0 0 1" />
+         <limit lower="0" upper="2.6" effort="0" velocity="0.5" />
+      </joint>
+      <joint name="${prefix}gripper_prismatic_joint_1" type="prismatic">
          <origin xyz="0 0 0" rpy="0 0 0" />
          <parent link="${prefix}gripper_rail_link" />
          <child link="${prefix}gripper_1_link" />
-         <axis xyz="0 1 0" />
+         <axis xyz="0 -1 0" />
          <limit lower="0" upper="0.027" effort="0" velocity="0.5" />
       </joint>
-      <joint name="${prefix}joint_8" type="prismatic">
+      <joint name="${prefix}gripper_prismatic_joint_2" type="prismatic">
          <origin xyz="0 0 0" rpy="0 0 0" />
          <parent link="${prefix}gripper_rail_link" />
          <child link="${prefix}gripper_2_link" />
-         <mimic joint="${prefix}joint_7" />
-         <axis xyz="0 -1 0" />
+         <mimic joint="${prefix}gripper_prismatic_joint_1" />
+         <axis xyz="0 1 0" />
          <limit lower="0" upper="0.027" effort="0" velocity="0.5" />
       </joint>
@@ -300,5 +309,5 @@
  <transmission name="tran6">
     <type>transmission_interface/SimpleTransmission</type>
-    <joint name="joint_7"/>
+    <joint name="gripper_prismatic_joint_1"/>
     <actuator name="motor6">
       <hardwareInterface>EffortJointInterface</hardwareInterface>

Commit message: Deleted gripper

File: widowx_arm_description/urdf/widowx.urdf.xacro (robot description, xacro)
@@ -133,5 +133,5 @@
          </inertial>
       </link>
-      <link name="${prefix}gripper_rail_link">
+      <!--link name="${prefix}gripper_rail_link">
          <visual>
             <origin xyz="0 0 0" rpy="0 0 1.57" />
@@ -194,5 +194,5 @@
             <inertia ixx="1.0" ixy="0.0" ixz="0.0" iyy="1.0" iyz="0.0" izz="1.0" />
          </inertial>
-      </link>
+      </link-->
       <!-- joints -->
       <joint name="${prefix}arm_base_joint" type="fixed">
@@ -237,5 +237,5 @@
          <limit lower="-2.617" upper="2.617" effort="0" velocity="1.571" />
       </joint>
-      <joint name="${prefix}joint_6" type="fixed">
+      <!--joint name="${prefix}joint_6" type="fixed">
          <origin xyz = "0 0 ${M_SCALE*43}" rpy="0 0 0" />
          <parent link="${prefix}wrist_2_link" />
@@ -265,5 +265,5 @@
          <axis xyz="0 1 0" />
          <limit lower="0" upper="0.027" effort="0" velocity="0.5" />
-      </joint>
+      </joint-->
    </xacro:macro>
   <transmission name="tran1">
@@ -299,5 +299,5 @@
     </actuator>
   </transmission>
- <transmission name="tran5">
+ <!--transmission name="tran5">
     <type>transmission_interface/SimpleTransmission</type>
     <joint name="joint_6"/>
@@ -314,4 +314,4 @@
       <mechanicalReduction>1</mechanicalReduction>
     </actuator>
-  </transmission>
+  </transmission-->
 </robot>
